File: ESP12ESwitch/ESP12ESwitch.kicad_pcb (KiCad board)
At the start: 2 copper layers, 12 parts, among them J1 Conn_01x06_Socket, J2 Conn_01x01_Pin, J3 B2+, J4 B1-, J5 B2-, J6 B1+, U1 ESP12E

Commit message: started automation
Parts:
- added JP1: RST, Jumper:SolderJumper-2_P1.3mm_Open_Pad1.0x1.5mm, B.Cu at (110.1, 102.1)
- added JP2: BOOT, Jumper:SolderJumper-2_P1.3mm_Open_Pad1.0x1.5mm, B.Cu at (87.4, 102.1)
- added SW1: RST, Aliexpress:5mmButton, B.Cu at (110.2, 96.0)
- added SW2: BOOT, Aliexpress:5mmButton, B.Cu at (87.6, 94.4)
- C1, R1, R2, R3, R4: moved to B.Cu
- moved R2 36.4 mm to (111.3, 72.6)
- moved R1 28.6 mm to (104.5, 97.5), turned to 180 degrees
- moved R3 26.7 mm to (87.9, 110.2)
- moved C1 26.5 mm to (85.9, 106.2), turned to -90 degrees
- moved R4 23.2 mm to (89.4, 106.1), turned to -90 degrees
Connections:
- R1 pad 1: Net-(SW1-B) -> Net-(JP1-B)
Routing:
- net Net-(R2-Pad1): track 0.00 -> 12.6 mm
- net Net-(J3-Pin_1): track 23.5 -> 35.6 mm

Commit message: improved layout
Parts:
- moved R3 21.9 mm to (89.4, 88.4), turned to 90 degrees
- moved R1 15.8 mm to (111.3, 83.2), turned to -90 degrees
- moved R2 10.4 mm to (104.1, 80.3)
- moved JP2 9.15 mm to (87.7, 93.0)
- moved JP1 9.14 mm to (110.1, 93.0)
- moved R4 9.00 mm to (91.9, 97.4)
- moved C1 8.31 mm to (91.9, 100.6)
- moved SW2 4.64 mm to (87.9, 99.1)
- moved SW1 3.05 mm to (110.2, 99.1)
Connections:
- U1 pad RESET: Net-(SW1-B) -> Net-(JP1-B)
Routing:
- net Net-(J1-Pin_1): track 32.4 -> 97.9 mm
- net Net-(J2-Pin_1): track 0.00 -> 58.8 mm
- net Net-(JP1-B): track 0.00 -> 32.8 mm
- net Net-(JP2-A): track 0.00 -> 18.5 mm
- net Net-(J3-Pin_1): track 35.6 -> 46.1 mm
- net Net-(R2-Pad1): track 12.6 -> 4.86 mm
- net Net-(R3-Pad2): track 0.00 -> 2.49 mm
Other:
- board outline added: 31.5 x 61 mm

Commit message: finalised layout, added cu fill
Connections:
- net Net-(J3-Pin_1) renamed /3V
- C1 pad 2: Net-(J1-Pin_1) -> /GND
- J1 pad 1: Net-(J1-Pin_1) -> /GND
- J4 pad 1: Net-(J1-Pin_1) -> /GND
- JP1 pad 1: Net-(J1-Pin_1) -> /GND
- JP2 pad 2: Net-(J1-Pin_1) -> /GND
- R3 pad 1: Net-(J1-Pin_1) -> /GND
- U1 pad GND: Net-(J1-Pin_1) -> /GND
Routing:
- net /3V: track 46.1 -> 87.9 mm
- net Net-(J1-Pin_1): track 97.9 -> 130.0 mm
- added copper zone on B.Cu, net /GND
Other:
- board size 31.5 x 61 mm -> 32 x 61 mm
