File: ESP12ESwitch/ESP12ESwitch.kicad_sch (KiCad schematic)
At the start: 14 parts, among them J1 Conn_01x06_Socket, J2 Conn_01x01_Pin, J3 B2+, J4 B1-, J5 B2-, J6 B1+, SW1 RST, SW2 BOOT, U1 ESP12E

Commit message: started automation
Parts:
- added JP1: RST, Jumper:SolderJumper-2_P1.3mm_Open_Pad1.0x1.5mm, symbol Jumper:SolderJumper_2_Open
- added JP2: BOOT, Jumper:SolderJumper-2_P1.3mm_Open_Pad1.0x1.5mm, symbol Jumper:SolderJumper_2_Open
- J1: footprint Connector_PinHeader_2.54mm:PinHeader_1x06_P2.54mm_Vertical_SMD_Pin1Left -> Connector_PinHeader_2.54mm:PinHeader_1x06_P2.54mm_Vertical
Connections:
- net at C1.2, J1.1 (Pin_1), J4.1 (Pin_1)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: now also JP1.1 (A), JP2.2 (B)
- net at SW1.2 (B), U1.RESET: no longer R1.1
- net at R4.1, SW2.1 (A), U1.GPIO0: now also JP2.1 (A)
- new net: JP1.2 (B), R1.1
Changed lines of the file:
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@@
   (junction (at 149.86 82.55) (diameter 0) (color 0 0 0 0)
   )
-  (junction (at 105.41 72.39) (diameter 0) (color 0 0 0 0)
+  (junction (at 87.63 72.39) (diameter 0) (color 0 0 0 0)
+  )
+  (junction (at 151.13 82.55) (diameter 0) (color 0 0 0 0)
   )
   (junction (at 83.82 77.47) (diameter 0) (color 0 0 0 0)
@@
   (junction (at 142.24 106.68) (diameter 0) (color 0 0 0 0)
   )
+  (junction (at 161.29 86.36) (diameter 0) (color 0 0 0 0)
+  )
   (junction (at 86.36 107.95) (diameter 0) (color 0 0 0 0)
   )
@@
     (stroke (width 0) (type default))
   )
-  (wire (pts (xy 78.74 72.39) (xy 93.98 72.39))
-    (stroke (width 0) (type default))
-  )
   (wire (pts (xy 144.78 74.93) (xy 142.24 74.93))
     (stroke (width 0) (type default))
   )
+  (wire (pts (xy 161.29 86.36) (xy 161.29 109.22))
+    (stroke (width 0) (type default))
+  )
+  (wire (pts (xy 95.25 67.31) (xy 87.63 67.31))
+    (stroke (width 0) (type default))
+  )
   (wire (pts (xy 83.82 77.47) (xy 87.63 77.47))
     (stroke (width 0) (type default))
   )
+  (wire (pts (xy 87.63 72.39) (xy 93.98 72.39))
+    (stroke (width 0) (type default))
+  )
   (wire (pts (xy 173.99 81.28) (xy 173.99 71.12))
     (stroke (width 0) (type default))
@@
     (stroke (width 0) (type default))
   )
+  (wire (pts (xy 158.75 86.36) (xy 161.29 86.36))
+    (stroke (width 0) (type default))
+  )
   (wire (pts (xy 78.74 72.39) (xy 78.74 107.95))
     (stroke (width 0) (type default))
@@
     (stroke (width 0) (type default))
   )
-  (wire (pts (xy 161.29 82.55) (xy 161.29 109.22))
+  (wire (pts (xy 161.29 82.55) (xy 161.29 86.36))
     (stroke (width 0) (type default))
   )
@@
     (stroke (width 0) (type default))
   )
+  (wire (pts (xy 87.63 67.31) (xy 87.63 72.39))
+    (stroke (width 0) (type default))
+  )
   (wire (pts (xy 109.22 90.17) (xy 96.52 90.17))
     (stroke (width 0) (type default))
@@
     (stroke (width 0) (type default))
   )
+  (wire (pts (xy 95.25 62.23) (xy 95.25 67.31))
+    (stroke (width 0) (type default))
+  )
+  (wire (pts (xy 78.74 72.39) (xy 87.63 72.39))
+    (stroke (width 0) (type default))
+  )
   (wire (pts (xy 86.36 102.87) (xy 86.36 107.95))
     (stroke (width 0) (type default))
   )
+  (wire (pts (xy 104.14 72.39) (xy 109.22 72.39))
+    (stroke (width 0) (type default))
+  )
   (wire (pts (xy 69.85 74.93) (xy 109.22 74.93))
     (stroke (width 0) (type default))
@@
     (stroke (width 0) (type default))
   )
+  (wire (pts (xy 102.87 62.23) (xy 102.87 69.85))
+    (stroke (width 0) (type default))
+  )
   (wire (pts (xy 66.04 97.79) (xy 66.04 107.95))
     (stroke (width 0) (type default))
   )
-  (wire (pts (xy 109.22 72.39) (xy 105.41 72.39))
-    (stroke (width 0) (type default))
-  )
   (wire (pts (xy 83.82 59.69) (xy 83.82 77.47))
     (stroke (width 0) (type default))
@@
     (stroke (width 0) (type default))
   )
-  (wire (pts (xy 105.41 67.31) (xy 105.41 72.39))
+  (wire (pts (xy 105.41 67.31) (xy 105.41 69.85))
+    (stroke (width 0) (type default))
+  )
+  (wire (pts (xy 102.87 69.85) (xy 105.41 69.85))
     (stroke (width 0) (type default))
   )
@@
     (stroke (width 0) (type default))
   )
-  (wire (pts (xy 105.41 72.39) (xy 104.14 72.39))
-    (stroke (width 0) (type default))
-  )
   (wire (pts (xy 96.52 104.14) (xy 99.06 104.14))
+    (stroke (width 0) (type default))
+  )
+  (wire (pts (xy 151.13 86.36) (xy 151.13 82.55))
     (stroke (width 0) (type default))
   )
@@
       (effects (font (size 1.27 1.27)) (justify left))
     )
-    (property "Footprint" "Connector_PinHeader_2.54mm:PinHeader_1x06_P2.54mm_Vertical_SMD_Pin1Left" (at 185.42 78.74 0)
+    (property "Footprint" "Connector_PinHeader_2.54mm:PinHeader_1x06_P2.54mm_Vertical" (at 185.42 78.74 0)
       (effects (font (size 1.27 1.27)) hide)
     )
@@
         (path "/f2cae78e-9019-4592-aebb-8554231d195c"
           (reference "J2") (unit 1)
+        )
+      )
+    )
+  )
+  (symbol (lib_id "Jumper:SolderJumper_2_Open") (at 99.06 62.23 0) (unit 1)
+    (in_bom yes) (on_board yes) (dnp no) (fields_autoplaced)
+    (property "Reference" "JP1" (at 99.06 55.88 0)
+      (effects (font (size 1.27 1.27)))
+    )
+    (property "Value" "RST" (at 99.06 58.42 0)
+      (effects (font (size 1.27 1.27)))
+    )
+    (property "Footprint" "Jumper:SolderJumper-2_P1.3mm_Open_Pad1.0x1.5mm" (at 99.06 62.23 0)
+      (effects (font (size 1.27 1.27)) hide)
+    )
+    (property "Datasheet" "~" (at 99.06 62.23 0)
+      (effects (font (size 1.27 1.27)) hide)
+    )
+    (pin "2")
+    (pin "1")
+    (instances
+      (project "ESP12ESwitch"
+        (path "/f2cae78e-9019-4592-aebb-8554231d195c"
+          (reference "JP1") (unit 1)
+        )
+      )
+    )
+  )
+  (symbol (lib_id "Jumper:SolderJumper_2_Open") (at 154.94 86.36 0) (unit 1)
+    (in_bom yes) (on_board yes) (dnp no) (fields_autoplaced)
+    (property "Reference" "JP2" (at 154.94 80.01 0)
+      (effects (font (size 1.27 1.27)))
+    )
+    (property "Value" "BOOT" (at 154.94 82.55 0)
+      (effects (font (size 1.27 1.27)))
+    )
+    (property "Footprint" "Jumper:SolderJumper-2_P1.3mm_Open_Pad1.0x1.5mm" (at 154.94 86.36 0)
+      (effects (font (size 1.27 1.27)) hide)
+    )
+    (property "Datasheet" "~" (at 154.94 86.36 0)
+      (effects (font (size 1.27 1.27)) hide)
+    )
+    (pin "2")
+    (pin "1")
+    (instances
+      (project "ESP12ESwitch"
+        (path "/f2cae78e-9019-4592-aebb-8554231d195c"
+          (reference "JP2") (unit 1)
         )
       )
@@
   )
   (symbol (lib_id "Device:R") (at 91.44 77.47 270) (unit 1)
-    (in_bom yes) (on_board yes) (dnp no) (fields_autoplaced)
+    (in_bom yes) (on_board yes) (dnp no)
     (property "Reference" "R2" (at 91.44 71.12 90)
       (effects (font (size 1.27 1.27)))

Commit message: improved layout
Connections:
- net at JP1.2 (B), R1.1: now also SW1.2 (B), U1.RESET
Changed lines of the file:
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@@
   (junction (at 149.86 82.55) (diameter 0) (color 0 0 0 0)
+  )
+  (junction (at 109.22 72.39) (diameter 0) (color 0 0 0 0)
   )
   (junction (at 87.63 72.39) (diameter 0) (color 0 0 0 0)
@@
   )
   (junction (at 96.52 90.17) (diameter 0) (color 0 0 0 0)
+  )
+  (junction (at 105.41 69.85) (diameter 0) (color 0 0 0 0)
   )
   (junction (at 142.24 106.68) (diameter 0) (color 0 0 0 0)
@@
     (stroke (width 0) (type default))
   )
+  (wire (pts (xy 109.22 69.85) (xy 109.22 72.39))
+    (stroke (width 0) (type default))
+  )
   (wire (pts (xy 142.24 69.85) (xy 142.24 72.39))
     (stroke (width 0) (type default))
@@
     (stroke (width 0) (type default))
   )
-  (wire (pts (xy 104.14 72.39) (xy 109.22 72.39))
-    (stroke (width 0) (type default))
-  )
   (wire (pts (xy 69.85 74.93) (xy 109.22 74.93))
     (stroke (width 0) (type default))
   )
   (wire (pts (xy 92.71 90.17) (xy 96.52 90.17))
+    (stroke (width 0) (type default))
+  )
+  (wire (pts (xy 105.41 69.85) (xy 109.22 69.85))
     (stroke (width 0) (type default))
   )
@@
     (stroke (width 0) (type default))
   )
+  (wire (pts (xy 104.14 72.39) (xy 109.22 72.39))
+    (stroke (width 0) (type default))
+  )

Commit message: finalised layout, added cu fill
Connections:
- net GND: now reaches C1.2, J1.1 (Pin_1), J4.1 (Pin_1), JP1.1 (A), JP2.2 (B), R3.1, SW1.1 (A), SW2.2 (B), U1.GND
- net 3V: now reaches C1.1, J3.1 (Pin_1), R1.2, R2.2, R4.2, U1.VCC
Changed lines of the file:
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@@
     (stroke (width 0) (type default))
+  )
+  (label "GND" (at 142.24 116.84 0) (fields_autoplaced)
+    (effects (font (size 1.27 1.27)) (justify left bottom))
+  )
+  (label "3V" (at 87.63 90.17 0) (fields_autoplaced)
+    (effects (font (size 1.27 1.27)) (justify left bottom))
   )
   (symbol (lib_id "Connector:Conn_01x06_Socket") (at 185.42 78.74 0) (unit 1)
