File: ESP32QuadSwitch/ESP32QuadSwitch/ESP32QuadSwitch.kicad_sch (KiCad schematic)
At the start: 13 parts, among them J1 Conn_01x01_Pin, J2 Conn_01x01_Pin, J3 Conn_01x01_Pin, J4 Conn_01x01_Pin, J5 Conn_01x06_Pin, J6 B2+, J7 B1-, J8 B1+, J9 B2-, U1 ESP32-S2-WROVER

Commit message: new PCB with esp32-s2
Parts:
- J1, J2, J3, J4: footprint (none) -> MountingHole:MountingHole_3.2mm_M3_DIN965_Pad
Changed lines of the file:
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@@
 			)
 		)
-		(property "Footprint" ""
+		(property "Footprint" "MountingHole:MountingHole_3.2mm_M3_DIN965_Pad"
 			(at 119.38 82.55 0)
 			(effects
@@
 			)
 		)
-		(property "Footprint" ""
+		(property "Footprint" "MountingHole:MountingHole_3.2mm_M3_DIN965_Pad"
 			(at 119.38 74.93 0)
 			(effects
@@
 			)
 		)
-		(property "Footprint" ""
+		(property "Footprint" "MountingHole:MountingHole_3.2mm_M3_DIN965_Pad"
 			(at 119.38 67.31 0)
 			(effects
@@
 			)
 		)
-		(property "Footprint" ""
+		(property "Footprint" "MountingHole:MountingHole_3.2mm_M3_DIN965_Pad"
 			(at 119.38 90.17 0)
 			(effects
